Commit message: smaller collision model

File: jsk_arc2017_baxter/robots/left_vacuum_gripper.xacro (robot description, xacro)
@@ -40,6 +40,6 @@
   <xacro:property name="lg_base_rect_offset_x" value="0.0065" />
   <xacro:property name="lg_base_rect_l" value="0.2805" />
-  <xacro:property name="lg_base_rect_h" value="0.107" />
-  <xacro:property name="lg_base_rect_w" value="0.15" />
+  <xacro:property name="lg_base_rect_h" value="0.05" />
+  <xacro:property name="lg_base_rect_w" value="0.05" />
   <xacro:property name="lg_camera_rect_offset_x" value="-0.061" />
   <xacro:property name="lg_camera_rect_offset_y" value="0.037" />
@@ -53,5 +53,5 @@
   <xacro:property name="lg_tube_rect_l" value="0.29" />
   <xacro:property name="lg_tube_rect_h" value="0.034" />
-  <xacro:property name="lg_tube_rect_w" value="0.081" />
+  <xacro:property name="lg_tube_rect_w" value="0.05" />
   <xacro:property name="lg_pad_with_base_offset_x" value="-0.048" />
   <xacro:property name="lg_pad_with_base_offset_y" value="0.0005" />
@@ -64,7 +64,7 @@
   <xacro:property name="lg_finger_base_rect_h" value="0.032" />
   <xacro:property name="lg_finger_base_rect_w" value="0.036" />
-  <xacro:property name="lg_finger_rect_l" value="0.04" />
-  <xacro:property name="lg_finger_rect_h" value="0.016" />
-  <xacro:property name="lg_finger_rect_w" value="0.11" />
+  <xacro:property name="lg_finger_rect_l" value="0.001" />
+  <xacro:property name="lg_finger_rect_h" value="0.001" />
+  <xacro:property name="lg_finger_rect_w" value="0.001" />
   <!--Joints-->
   <xacro:property name="lg_hand_offset_x" value="-0.01" />

File: jsk_arc2017_baxter/robots/right_vacuum_gripper.xacro (robot description, xacro)
@@ -40,6 +40,6 @@
   <xacro:property name="rg_base_rect_offset_x" value="0.0065" />
   <xacro:property name="rg_base_rect_l" value="0.2805" />
-  <xacro:property name="rg_base_rect_h" value="0.107" />
-  <xacro:property name="rg_base_rect_w" value="0.15" />
+  <xacro:property name="rg_base_rect_h" value="0.05" />
+  <xacro:property name="rg_base_rect_w" value="0.05" />
   <xacro:property name="rg_camera_rect_offset_x" value="-0.061" />
   <xacro:property name="rg_camera_rect_offset_y" value="-0.037" />
@@ -53,5 +53,5 @@
   <xacro:property name="rg_tube_rect_l" value="0.29" />
   <xacro:property name="rg_tube_rect_h" value="0.034" />
-  <xacro:property name="rg_tube_rect_w" value="0.081" />
+  <xacro:property name="rg_tube_rect_w" value="0.05" />
   <xacro:property name="rg_pad_with_base_offset_x" value="-0.048" />
   <xacro:property name="rg_pad_with_base_offset_y" value="-0.0005" />
@@ -64,7 +64,7 @@
   <xacro:property name="rg_finger_base_rect_h" value="0.032" />
   <xacro:property name="rg_finger_base_rect_w" value="0.036" />
-  <xacro:property name="rg_finger_rect_l" value="0.04" />
-  <xacro:property name="rg_finger_rect_h" value="0.016" />
-  <xacro:property name="rg_finger_rect_w" value="0.11" />
+  <xacro:property name="rg_finger_rect_l" value="0.001" />
+  <xacro:property name="rg_finger_rect_h" value="0.001" />
+  <xacro:property name="rg_finger_rect_w" value="0.001" />
   <!--Joints-->
   <xacro:property name="rg_hand_offset_x" value="-0.01" />
